Commit message: Markers/subscribers for transformation

File: environment/models/narkin/narkin.urdf (robot description, URDF)
Before this commit: robot Narkin, 10 links, 9 joints
Joints:
- removed joint Actuator0
- added joint joint_8: type fixed, parent narko_base_link, child base_link, origin xyz=0 0 0.15 rpy=0 0 0
